File: keyboard.kicad_pcb (KiCad board)
At the start: 2 copper layers, 27 parts, among them J1 USB4085-GF-A_REVB, SW2 SW_Push, SW3 SW_Push, SW4 SW_Push, SW5 SW_Push, U1 ATmega32U4-A, Y1 Crystal_GND24_Small

Commit message: V1
Parts:
- removed F1: 500mA, Fuse:Fuse_1206_3216Metric
- removed J1: USB4085-GF-A_REVB, USB-C:GCT_USB4085-GF-A_REVB
- removed R5, R6: 5.1k, Resistor_SMD:R_0805_2012Metric
- removed S1: 8-1437565-1, Button:SW_8-1437565-1
- removed SW2, SW3, SW4, SW5: SW_Push, MX_keys:MX-Hotswap-1U
- added 5V+2: Power, TestPoint:TestPoint_Pad_1.0x1.0mm, B.Cu at (247.8, 77.0)
- added Custom-1: SW_Push, MX_keys:MX-Hotswap-1U, B.Cu at (256.4, 69.8)
- added Custom-2: SW_Push, MX_keys:MX-Hotswap-1U, B.Cu at (256.4, 88.9)
- added Custom-3: SW_Push, MX_keys:MX-Hotswap-1U, B.Cu at (256.4, 108.0)
- added Custom-4: SW_Push, MX_keys:MX-Hotswap-1U, B.Cu at (256.4, 127.0)
- added Custom-5: SW_Push, MX_keys:MX-Hotswap-1U, B.Cu at (256.4, 146.1)
- added D+1: D+, TestPoint:TestPoint_Pad_1.0x1.0mm, B.Cu at (242.9, 77.0)
- added D-1: D-, TestPoint:TestPoint_Pad_1.0x1.0mm, B.Cu at (236.5, 71.4)
- added D10: D_Small, Diode_SMD:D_SOD-123, B.Cu at (198.4, 90.5)
- added D11: D_Small, Diode_SMD:D_SOD-123, B.Cu at (217.5, 71.4)
- added D12: D_Small, Diode_SMD:D_SOD-123, B.Cu at (217.5, 92.1)
- added D13: D_Small, Diode_SMD:D_SOD-123, B.Cu at (198.4, 109.5)
- added D14: D_Small, Diode_SMD:D_SOD-123, B.Cu at (198.4, 128.6)
- added D16: D_Small, Diode_SMD:D_SOD-123, B.Cu at (217.5, 130.2)
- added D17: D_Small, Diode_SMD:D_SOD-123, B.Cu at (251.6, 73.8)
- added D18: D_Small, Diode_SMD:D_SOD-123, B.Cu at (248.4, 90.5)
- added D19: D_Small, Diode_SMD:D_SOD-123, B.Cu at (249.2, 110.3)
- added D20: D_Small, Diode_SMD:D_SOD-123, B.Cu at (248.4, 128.5)
- added D21: D_Small, Diode_SMD:D_SOD-123, B.Cu at (169.9, 147.6)
- added D23: D_Small, Diode_SMD:D_SOD-123, B.Cu at (198.4, 147.6)
- added D25: D_Small, Diode_SMD:D_SOD-123, B.Cu at (248.4, 147.6)
- added D5: D_Small, Diode_SMD:D_SOD-123, B.Cu at (160.3, 109.5)
- added D6: D_Small, Diode_SMD:D_SOD-123, B.Cu at (160.3, 128.6)
- added D7: D_Small, Diode_SMD:D_SOD-123, B.Cu at (179.4, 109.5)
- added D8: D_Small, Diode_SMD:D_SOD-123, B.Cu at (179.4, 128.6)
- added D9: D_Small, Diode_SMD:D_SOD-123, B.Cu at (198.4, 71.4)
- added F2: 500mA, Fuse:Fuse_1206_3216Metric, B.Cu at (244.5, 73.6)
- added GND1: Power, TestPoint:TestPoint_Pad_1.0x1.0mm, B.Cu at (247.9, 72.4)
- added J2: TYPE-C-31-M-12, USB-C:HRO_TYPE-C-31-M-12, B.Cu at (241.1, 61.8)
- added Key_*1: SW_Push, MX_keys:MX-Hotswap-1U, B.Cu at (206.4, 69.8)
- added Key_+1: SW_Push_U2, Button_Switch_Keyboard:MX-Hotswap-2U-Vertical-ReversedStabilizers, B.Cu at (225.4, 98.4)
- added Key_-1: SW_Push, MX_keys:MX-Hotswap-1U, B.Cu at (225.4, 69.8)
- added Key_/1: SW_Push, MX_keys:MX-Hotswap-1U, B.Cu at (187.3, 69.8)
- added Key_0: SW_Push_U2, Button_Switch_Keyboard:MX-Hotswap-2U-ReversedStabilizers, B.Cu at (177.8, 146.1)
- added Key_1: SW_Push, MX_keys:MX-Hotswap-1U, B.Cu at (168.3, 127.0)
- added Key_2: SW_Push, MX_keys:MX-Hotswap-1U, B.Cu at (187.3, 127.0)
- added Key_3: SW_Push, MX_keys:MX-Hotswap-1U, B.Cu at (206.4, 127.0)
- added Key_4: SW_Push, MX_keys:MX-Hotswap-1U, B.Cu at (168.3, 108.0)
- added Key_5: SW_Push, MX_keys:MX-Hotswap-1U, B.Cu at (187.3, 108.0)
- added Key_6: SW_Push, MX_keys:MX-Hotswap-1U, B.Cu at (206.4, 108.0)
- added Key_7: SW_Push, MX_keys:MX-Hotswap-1U, B.Cu at (168.3, 88.9)
- added Key_8: SW_Push, MX_keys:MX-Hotswap-1U, B.Cu at (187.3, 88.9)
- added Key_9: SW_Push, MX_keys:MX-Hotswap-1U, B.Cu at (206.4, 88.9)
- added Key_del1: SW_Push, MX_keys:MX-Hotswap-1U, B.Cu at (206.4, 146.1)
- added Key_enter1: SW_Push_U2, Button_Switch_Keyboard:MX-Hotswap-2U-Vertical-ReversedStabilizers, B.Cu at (225.4, 136.5)
- added NumLock1: SW_Push, MX_keys:MX-Hotswap-1U, B.Cu at (168.3, 69.8)
- added R7: 5.1k, Resistor_SMD:R_0805_2012Metric, B.Cu at (244.6, 69.1)
- added R8: 5.1k, Resistor_SMD:R_0805_2012Metric, B.Cu at (236.7, 69.1)
- added S2: TS-1187A-B-A-B, USB-C:SW_TS-1187A-B-A-B, B.Cu at (240.5, 130.2)
- added TV1: ~, Button_Switch_Keyboard:SOT-23-6_L2.9-W1.6-P0.95-LS2.8-BR, B.Cu at (240.5, 70.1)
- R1: moved to B.Cu
- moved C8 105.1 mm to (245.4, 112.7), turned to 0 degrees
- moved C5 97.9 mm to (245.4, 110.3)
- moved C1 97.8 mm to (254.2, 99.8), turned to 0 degrees
- moved Y1 97.6 mm to (241.4, 110.3), turned to 0 degrees
- moved C2 94.5 mm to (233.4, 105.7)
- moved R1 94.4 mm to (233.4, 97.0)
- moved C3 94.3 mm to (237.2, 92.1)
- moved U1 93.6 mm to (241.2, 101.6)
- moved C4 93.1 mm to (249.2, 97.5)
- moved R2 91.8 mm to (241.0, 73.9), turned to 90 degrees
- moved C7 90.5 mm to (237.8, 110.2), turned to -90 degrees
- moved R4 90.3 mm to (241.2, 125.4), turned to 0 degrees
- moved C6 89.0 mm to (244.3, 93.7), turned to 0 degrees
- moved R3 84.3 mm to (239.0, 73.9), turned to -90 degrees
- moved D4 19.7 mm to (179.4, 90.4), turned to 90 degrees
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Connections:
- U1 pad 10: Y0 -> unconnected-(U1-PB2-Pad10)
- U1 pad 11: Y1 -> unconnected-(U1-PB3-Pad11)
- U1 pad 26: unconnected-(U1-PD6-Pad26) -> Y3
- U1 pad 27: unconnected-(U1-PD7-Pad27) -> Y2
- U1 pad 28: unconnected-(U1-PB4-Pad28) -> Y1
- U1 pad 29: unconnected-(U1-PB5-Pad29) -> Y0
- U1 pad 36: unconnected-(U1-PF7-Pad36) -> X0
- U1 pad 37: unconnected-(U1-PF6-Pad37) -> X1
- U1 pad 38: unconnected-(U1-PF5-Pad38) -> X4
- U1 pad 39: unconnected-(U1-PF4-Pad39) -> X3
- U1 pad 40: unconnected-(U1-PF1-Pad40) -> X2
- U1 pad 8: X0 -> unconnected-(U1-PB0-Pad8)
- U1 pad 9: X1 -> Y4
Routing:
- net X4: track 0.00 -> 140.3 mm, vias 0 -> 2
- net X3: track 0.00 -> 130.7 mm, vias 0 -> 2
- net Y0: track 28.6 -> 154.7 mm, vias 1 -> 5
- net X2: track 0.00 -> 113.2 mm, vias 0 -> 3
- net Y2: track 0.00 -> 108.8 mm, vias 0 -> 5
- net Y4: track 0.00 -> 105.1 mm, vias 0 -> 5
- net GND: track 84.0 -> 170.0 mm, vias 2 -> 4
- net Y3: track 0.00 -> 79.1 mm, vias 0 -> 4
- net X0: track 53.5 -> 115.6 mm, vias 2 -> 3
- net Y1: track 49.5 -> 109.7 mm, vias 1 -> 4
- net X1: track 51.2 -> 100.9 mm, vias 2 -> 3
- net Net-(J1-CC2): track 24.7 -> 0.00 mm
- net Net-(U1-XTAL1): track 23.2 -> 4.62 mm, vias 2 -> 0
- net Net-(U1-D-): track 16.1 -> 32.7 mm, vias 2 -> 0
- net Net-(U1-D+): track 16.5 -> 32.9 mm, vias 2 -> 0
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Other:
- board outline added: 108.2 x 96.2 mm
